File: pcb/mls25.kicad_sch (KiCad schematic)
At the start: 6 parts

Commit message: Rename `mls12` to `mls25`
Module output was changed from 12W to 25W during the course of development.
Update filenames to reflect that.
Other:
- sheet BUCK 3V3: file mls12_buck_3v3.kicad_sch -> mls25_buck_3v3.kicad_sch
- sheet ETH-CONN: file mls12_eth_conn.kicad_sch -> mls25_eth_conn.kicad_sch
- sheet ETH-PHY: file mls12_eth_phy.kicad_sch -> mls25_eth_phy.kicad_sch
- sheet ETH-PoE+: file mls12_eth_poe.kicad_sch -> mls25_eth_poe.kicad_sch
- sheet LED output 1: file mls12_led_output.kicad_sch -> mls25_led_output.kicad_sch
- sheet LED output 2: file mls12_led_output.kicad_sch -> mls25_led_output.kicad_sch
- sheet MCU: file mls12_mcu.kicad_sch -> mls25_mcu.kicad_sch
- sheet NOR Flash: file mls12_nor_flash.kicad_sch -> mls25_nor_flash.kicad_sch
Changed lines of the file:
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@@
 		)
 		(instances
-			(project "mls12"
+			(project "mls25"
 				(path "/53bda2f8-fdf0-44f4-aced-3b46017d299c"
 					(reference "FID2")
@@
 		)
 		(instances
-			(project "mls12"
+			(project "mls25"
 				(path "/53bda2f8-fdf0-44f4-aced-3b46017d299c"
 					(reference "H3")
@@
 		)
 		(instances
-			(project "mls12"
+			(project "mls25"
 				(path "/53bda2f8-fdf0-44f4-aced-3b46017d299c"
 					(reference "H2")
@@
 		)
 		(instances
-			(project "mls12"
+			(project "mls25"
 				(path "/53bda2f8-fdf0-44f4-aced-3b46017d299c"
 					(reference "FID3")
@@
 			)
 		)
-		(property "Sheetfile" "mls12_nor_flash.kicad_sch"
+		(property "Sheetfile" "mls25_nor_flash.kicad_sch"
 			(at 187.96 105.9946 0)
 			(effects
@@
 		)
 		(instances
-			(project "mls12"
+			(project "mls25"
 				(path "/53bda2f8-fdf0-44f4-aced-3b46017d299c"
 					(page "7")
@@
 			)
 		)
-		(property "Sheetfile" "mls12_mcu.kicad_sch"
+		(property "Sheetfile" "mls25_mcu.kicad_sch"
 			(at 148.59 133.9346 0)
 			(effects
@@
 		)
 		(instances
-			(project "mls12"
+			(project "mls25"
 				(path "/53bda2f8-fdf0-44f4-aced-3b46017d299c"
 					(page "6")
@@
 			)
 		)
-		(property "Sheetfile" "mls12_led_output.kicad_sch"
+		(property "Sheetfile" "mls25_led_output.kicad_sch"
 			(at 187.96 119.9646 0)
 			(effects
@@
 		)
 		(instances
-			(project "mls12"
+			(project "mls25"
 				(path "/53bda2f8-fdf0-44f4-aced-3b46017d299c"
 					(page "8")
@@
 			)
 		)
-		(property "Sheetfile" "mls12_eth_poe.kicad_sch"
+		(property "Sheetfile" "mls25_eth_poe.kicad_sch"
 			(at 109.22 86.9446 0)
 			(effects
@@
 		)
 		(instances
-			(project "mls12"
+			(project "mls25"
 				(path "/53bda2f8-fdf0-44f4-aced-3b46017d299c"
 					(page "3")
@@
 			)
 		)
-		(property "Sheetfile" "mls12_buck_3v3.kicad_sch"
+		(property "Sheetfile" "mls25_buck_3v3.kicad_sch"
 			(at 148.59 86.9446 0)
 			(effects
@@
 		)
 		(instances
-			(project "mls12"
+			(project "mls25"
 				(path "/53bda2f8-fdf0-44f4-aced-3b46017d299c"
 					(page "5")
@@
 			)
 		)
-		(property "Sheetfile" "mls12_eth_conn.kicad_sch"
+		(property "Sheetfile" "mls25_eth_conn.kicad_sch"
 			(at 78.74 119.9646 0)
 			(effects
@@
 		)
 		(instances
-			(project "mls12"
+			(project "mls25"
 				(path "/53bda2f8-fdf0-44f4-aced-3b46017d299c"
 					(page "2")
@@
 			)
 		)
-		(property "Sheetfile" "mls12_led_output.kicad_sch"
+		(property "Sheetfile" "mls25_led_output.kicad_sch"
 			(at 187.96 133.9346 0)
 			(effects
@@
 		)
 		(instances
-			(project "mls12"
+			(project "mls25"
 				(path "/53bda2f8-fdf0-44f4-aced-3b46017d299c"
 					(page "9")
@@
 			)
 		)
-		(property "Sheetfile" "mls12_eth_phy.kicad_sch"
+		(property "Sheetfile" "mls25_eth_phy.kicad_sch"
 			(at 109.22 119.9646 0)
 			(effects
@@
 		)
 		(instances
-			(project "mls12"
+			(project "mls25"
 				(path "/53bda2f8-fdf0-44f4-aced-3b46017d299c"
 					(page "4")
