File: pcb/mls25_eth_conn.kicad_sch (KiCad schematic)
At the start: 12 parts, among them J1 MTJ-88ARX1-FSM-LG

Commit message: Rename `mls12` to `mls25`
Module output was changed from 12W to 25W during the course of development.
Update filenames to reflect that.
Parts:
- D1, D2: symbol mls12:ESDS312DBV -> mls25:ESDS312DBV
- TR1: footprint mls12:7490120110 -> mls25:7490120110; symbol mls12:7490120110 -> mls25:7490120110
Changed lines of the file:
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@@
 		)
 		(instances
-			(project "mls12"
+			(project "mls25"
 				(path "/53bda2f8-fdf0-44f4-aced-3b46017d299c/cde1e0ff-e1f1-4d38-b939-7ba11eaafca9"
 					(reference "C2")
@@
 		)
 		(instances
-			(project "mls12"
+			(project "mls25"
 				(path "/53bda2f8-fdf0-44f4-aced-3b46017d299c/cde1e0ff-e1f1-4d38-b939-7ba11eaafca9"
 					(reference "R1")
@@
 		)
 		(instances
-			(project "mls12"
+			(project "mls25"
 				(path "/53bda2f8-fdf0-44f4-aced-3b46017d299c/cde1e0ff-e1f1-4d38-b939-7ba11eaafca9"
 					(reference "C3")
@@
 		)
 		(instances
-			(project "mls12"
+			(project "mls25"
 				(path "/53bda2f8-fdf0-44f4-aced-3b46017d299c/cde1e0ff-e1f1-4d38-b939-7ba11eaafca9"
 					(reference "J1")
@@
 		)
 		(instances
-			(project "mls12"
+			(project "mls25"
 				(path "/53bda2f8-fdf0-44f4-aced-3b46017d299c/cde1e0ff-e1f1-4d38-b939-7ba11eaafca9"
 					(reference "R3")
@@
 	)
 	(symbol
-		(lib_id "mls12:7490120110")
+		(lib_id "mls25:7490120110")
 		(at 163.83 95.25 180)
 		(unit 1)
@@
 			)
 		)
-		(property "Footprint" "mls12:7490120110"
+		(property "Footprint" "mls25:7490120110"
 			(at 163.83 82.55 0)
 			(effects
@@
 	)
 	(symbol
-		(lib_id "mls12:ESDS312DBV")
+		(lib_id "mls25:ESDS312DBV")
 		(at 210.82 104.14 270)
 		(unit 1)
@@
 		)
 		(instances
-			(project "mls12"
+			(project "mls25"
 				(path "/53bda2f8-fdf0-44f4-aced-3b46017d299c/cde1e0ff-e1f1-4d38-b939-7ba11eaafca9"
 					(reference "D2")
@@
 		)
 		(instances
-			(project "mls12"
+			(project "mls25"
 				(path "/53bda2f8-fdf0-44f4-aced-3b46017d299c/cde1e0ff-e1f1-4d38-b939-7ba11eaafca9"
 					(reference "#PWR01")
@@
 		)
 		(instances
-			(project "mls12"
+			(project "mls25"
 				(path "/53bda2f8-fdf0-44f4-aced-3b46017d299c/cde1e0ff-e1f1-4d38-b939-7ba11eaafca9"
 					(reference "R2")
@@
 		)
 		(instances
-			(project "mls12"
+			(project "mls25"
 				(path "/53bda2f8-fdf0-44f4-aced-3b46017d299c/cde1e0ff-e1f1-4d38-b939-7ba11eaafca9"
 					(reference "#PWR06")
@@
 	(symbol
 		(lib_name "ESDS312DBV_1")
-		(lib_id "mls12:ESDS312DBV")
+		(lib_id "mls25:ESDS312DBV")
 		(at 210.82 87.63 270)
 		(unit 1)
@@
 		)
 		(instances
-			(project "mls12"
+			(project "mls25"
 				(path "/53bda2f8-fdf0-44f4-aced-3b46017d299c/cde1e0ff-e1f1-4d38-b939-7ba11eaafca9"
 					(reference "D1")
@@
 		)
 		(instances
-			(project "mls12"
+			(project "mls25"
 				(path "/53bda2f8-fdf0-44f4-aced-3b46017d299c/cde1e0ff-e1f1-4d38-b939-7ba11eaafca9"
 					(reference "R5")
@@
 		)
 		(instances
-			(project "mls12"
+			(project "mls25"
 				(path "/53bda2f8-fdf0-44f4-aced-3b46017d299c/cde1e0ff-e1f1-4d38-b939-7ba11eaafca9"
 					(reference "#PWR05")
@@
 		)
 		(instances
-			(project "mls12"
+			(project "mls25"
 				(path "/53bda2f8-fdf0-44f4-aced-3b46017d299c/cde1e0ff-e1f1-4d38-b939-7ba11eaafca9"
 					(reference "R4")
@@
 		)
 		(instances
-			(project "mls12"
+			(project "mls25"
 				(path "/53bda2f8-fdf0-44f4-aced-3b46017d299c/cde1e0ff-e1f1-4d38-b939-7ba11eaafca9"
 					(reference "C1")
@@
 		)
 		(instances
-			(project "mls12"
+			(project "mls25"
 				(path "/53bda2f8-fdf0-44f4-aced-3b46017d299c/cde1e0ff-e1f1-4d38-b939-7ba11eaafca9"
 					(reference "#PWR02")
@@
 		)
 		(instances
-			(project "mls12"
+			(project "mls25"
 				(path "/53bda2f8-fdf0-44f4-aced-3b46017d299c/cde1e0ff-e1f1-4d38-b939-7ba11eaafca9"
 					(reference "#PWR03")

Commit message: Fix ERC warnings/errors
*  Add NC-flags to microcontroller pins.
*  Fix STM32 VCAP, ~RESET pin type.
*  Add PWR_FLAG symbols.
Changed lines of the file:
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@@
 	(title_block
 		(title "Ethernet RJ45 + Magnetics")
-		(date "2025-07-26")
+		(date "2025-09-27")
 		(rev "A")
 		(company "Quomodo BV")
@@
 	)
 	(junction
+		(at 77.47 105.41)
+		(diameter 0)
+		(color 0 0 0 0)
+	)
+	(junction
 		(at 204.47 93.98)
 		(diameter 0)
@@
 	(wire
 		(pts
-			(xy 77.47 104.14) (xy 77.47 107.95)
+			(xy 77.47 104.14) (xy 77.47 105.41)
 		)
 		(stroke
@@
 		(pts
 			(xy 205.74 90.17) (xy 204.47 90.17)
+		)
+		(stroke
+			(width 0)
+			(type default)
+		)
+	)
+	(wire
+		(pts
+			(xy 77.47 105.41) (xy 77.47 107.95)
 		)
 		(stroke
@@
 			)
 		)
+	)
+	(symbol
+		(lib_id "power:PWR_FLAG")
+		(at 77.47 105.41 270)
+		(unit 1)
+		(exclude_from_sim no)
+		(in_bom yes)
+		(on_board yes)
+		(dnp no)
+		(fields_autoplaced yes)
+		(property "Reference" "#FLG03"
+			(at 79.375 105.41 0)
+			(effects
+				(font
+					(size 1.27 1.27)
+				)
+				(hide yes)
+			)
+		)
+		(property "Value" "PWR_FLAG"
+			(at 81.28 105.4099 90)
+			(effects
+				(font
+					(size 1.27 1.27)
+				)
+				(justify left)
+				(hide yes)
+			)
+		)
+		(property "Footprint" ""
+			(at 77.47 105.41 0)
+			(effects
+				(font
+					(size 1.27 1.27)
+				)
+				(hide yes)
+			)
+		)
+		(property "Datasheet" "~"
+			(at 77.47 105.41 0)
+			(effects
+				(font
+					(size 1.27 1.27)
+				)
+				(hide yes)
+			)
+		)
+		(property "Description" "Special symbol for telling ERC where power comes from"
+			(at 77.47 105.41 0)
+			(effects
+				(font
+					(size 1.27 1.27)
+				)
+				(hide yes)
+			)
+		)
+		(property "MF" ""
+			(at 77.47 105.41 0)
+			(effects
+				(font
+					(size 1.27 1.27)
+				)
+				(hide yes)
+			)
+		)
+		(property "MPN" ""
+			(at 77.47 105.41 0)
+			(effects
+				(font
+					(size 1.27 1.27)
+				)
+				(hide yes)
+			)
+		)
+		(pin "1"
+		)
+		(instances
+			(project ""
+				(path "/53bda2f8-fdf0-44f4-aced-3b46017d299c/cde1e0ff-e1f1-4d38-b939-7ba11eaafca9"
+					(reference "#FLG03")
+					(unit 1)
+				)
+			)
+		)
