File: pcb/mls25_eth_phy.kicad_sch (KiCad schematic)
At the start: 27 parts, among them U2 KSZ8081RNA, Y1 25MHz

Commit message: Fix ERC warnings/errors
*  Add NC-flags to microcontroller pins.
*  Fix STM32 VCAP, ~RESET pin type.
*  Add PWR_FLAG symbols.
Changed lines of the file:
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@@
 	(title_block
 		(title "Ethernet PHY")
-		(date "2025-07-26")
+		(date "2025-09-27")
 		(rev "A")
 		(company "Quomodo BV")
@@
 					(unit 1)
 				)
+			)
+		)
+	)
+	(symbol
+		(lib_id "power:PWR_FLAG")
+		(at 135.89 43.18 0)
+		(unit 1)
+		(exclude_from_sim no)
+		(in_bom yes)
+		(on_board yes)
+		(dnp no)
+		(fields_autoplaced yes)
+		(property "Reference" "#FLG08"
+			(at 135.89 41.275 0)
+			(effects
+				(font
+					(size 1.27 1.27)
+				)
+				(hide yes)
+			)
+		)
+		(property "Value" "PWR_FLAG"
+			(at 135.89 38.1 0)
+			(effects
+				(font
+					(size 1.27 1.27)
+				)
+				(hide yes)
+			)
+		)
+		(property "Footprint" ""
+			(at 135.89 43.18 0)
+			(effects
+				(font
+					(size 1.27 1.27)
+				)
+				(hide yes)
+			)
+		)
+		(property "Datasheet" "~"
+			(at 135.89 43.18 0)
+			(effects
+				(font
+					(size 1.27 1.27)
+				)
+				(hide yes)
+			)
+		)
+		(property "Description" "Special symbol for telling ERC where power comes from"
+			(at 135.89 43.18 0)
+			(effects
+				(font
+					(size 1.27 1.27)
+				)
+				(hide yes)
+			)
+		)
+		(property "MF" ""
+			(at 135.89 43.18 0)
+			(effects
+				(font
+					(size 1.27 1.27)
+				)
+				(hide yes)
+			)
+		)
+		(property "MPN" ""
+			(at 135.89 43.18 0)
+			(effects
+				(font
+					(size 1.27 1.27)
+				)
+				(hide yes)
+			)
+		)
+		(pin "1"
+		)
+		(instances
+			(project ""
+				(path "/53bda2f8-fdf0-44f4-aced-3b46017d299c/f9d4ebc4-b22e-4ea3-9755-37111373d6cf"
+					(reference "#FLG08")
+					(unit 1)
+				)

Commit message: Tweaks/fixes after design review
*  Fix RJ45 refdes on silkscreen.
*  Change PHY IRQ pullup from 1K to 4K7 per datasheet recommendations.
*  Add skew correction on MDI TX differential pair.
*  Remove copper under magnetics.
*  Add annotation that TYP2_DET signal requires MCU internal pullup.
Parts:
- R13: value 1K -> 4K7; MPN AC0603JR-131KL -> RC0603JR-134K7L
Changed lines of the file:
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@@
 			)
 		)
-		(property "Value" "1K"
+		(property "Value" "4K7"
 			(at 215.9 110.4899 0)
 			(effects
@@
 			)
 		)
-		(property "Datasheet" "https://www.mouser.be/datasheet/2/447/PYu_AC_51_RoHS_L_11-3418659.pdf"
+		(property "Datasheet" "https://www.mouser.be/datasheet/2/447/YAGEO_PYu_RC_Group_51_RoHS_L_12-3313492.pdf"
 			(at 213.36 109.22 0)
 			(effects
@@
 			)
 		)
-		(property "MPN" "AC0603JR-131KL"
+		(property "MPN" "RC0603JR-134K7L"
 			(at 213.36 109.22 0)
 			(effects

Commit message: Change PHY to datasheet recommended footprint
Default footprint in the Kicad libraries for KSZ8081 deviates from the
datasheet recommendations. QFN parts can be fiddly, so it's best to stick
closely to the recommendations:

*  Pads are much shorter and a bit thinner.
*  Solder stencil openings for exposed pad are smaller, spaced out a bit less.
Parts:
- U2: footprint Package_DFN_QFN:QFN-24-1EP_4x4mm_P0.5mm_EP2.6x2.6mm -> mls25:KSZ8081_QFN-24-1EP_4x4mm_P0.5mm_EP2.6x2.6mm
Changed lines of the file:
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@@
 			)
 		)
-		(property "Footprint" "Package_DFN_QFN:QFN-24-1EP_4x4mm_P0.5mm_EP2.6x2.6mm"
+		(property "Footprint" "mls25:KSZ8081_QFN-24-1EP_4x4mm_P0.5mm_EP2.6x2.6mm"
 			(at 100.33 129.54 0)
 			(effects

Commit message: Exclude test pads from BOM
Parts:
- TP10, TP11, TP12, TP13, TP31, TP9: now left out of the parts list
Changed lines of the file:
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@@
 		(unit 1)
 		(exclude_from_sim no)
-		(in_bom yes)
+		(in_bom no)
 		(on_board yes)
 		(dnp no)
@@
 		(unit 1)
 		(exclude_from_sim no)
-		(in_bom yes)
+		(in_bom no)
 		(on_board yes)
 		(dnp no)
@@
 		(unit 1)
 		(exclude_from_sim no)
-		(in_bom yes)
+		(in_bom no)
 		(on_board yes)
 		(dnp no)
@@
 		(unit 1)
 		(exclude_from_sim no)
-		(in_bom yes)
+		(in_bom no)
 		(on_board yes)
 		(dnp no)
@@
 		(unit 1)
 		(exclude_from_sim no)
-		(in_bom yes)
+		(in_bom no)
 		(on_board yes)
 		(dnp no)
@@
 		(unit 1)
 		(exclude_from_sim no)
-		(in_bom yes)
+		(in_bom no)
 		(on_board yes)
 		(dnp no)
