File: pcb/mls25_eth_poe.kicad_sch (KiCad schematic)
At the start: 26 parts, among them U1 DPC817S-C-TR

Commit message: Rename `mls12` to `mls25`
Module output was changed from 12W to 25W during the course of development.
Update filenames to reflect that.
Parts:
- A1: footprint mls12:Ag5724-LPB -> mls25:Ag5724-LPB; symbol mls12:Ag5724-LPB -> mls25:Ag5724-LPB
- D3, D4: footprint mls12:LMB110S-TP -> mls25:LMB110S-TP; symbol mls12:LMB110S-TP -> mls25:LMB110S-TP
- U1: footprint mls12:DPC817S-C-TR -> mls25:DPC817S-C-TR
Changed lines of the file:
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@@
 		)
 		(instances
-			(project "mls12"
+			(project "mls25"
 				(path "/53bda2f8-fdf0-44f4-aced-3b46017d299c/9f8390ae-91ea-4278-be1f-a82b5834f728"
 					(reference "TP7")
@@
 	)
 	(symbol
-		(lib_id "mls12:LMB110S-TP")
+		(lib_id "mls25:LMB110S-TP")
 		(at 68.58 86.36 0)
 		(unit 1)
@@
 			)
 		)
-		(property "Footprint" "mls12:LMB110S-TP"
+		(property "Footprint" "mls25:LMB110S-TP"
 			(at 72.39 83.185 0)
 			(effects
@@
 		)
 		(instances
-			(project "mls12"
+			(project "mls25"
 				(path "/53bda2f8-fdf0-44f4-aced-3b46017d299c/9f8390ae-91ea-4278-be1f-a82b5834f728"
 					(reference "#PWR013")
@@
 		)
 		(instances
-			(project "mls12"
+			(project "mls25"
 				(path "/53bda2f8-fdf0-44f4-aced-3b46017d299c/9f8390ae-91ea-4278-be1f-a82b5834f728"
 					(reference "TP8")
@@
 		)
 		(instances
-			(project "mls12"
+			(project "mls25"
 				(path "/53bda2f8-fdf0-44f4-aced-3b46017d299c/9f8390ae-91ea-4278-be1f-a82b5834f728"
 					(reference "#PWR09")
@@
 		)
 		(instances
-			(project "mls12"
+			(project "mls25"
 				(path "/53bda2f8-fdf0-44f4-aced-3b46017d299c/9f8390ae-91ea-4278-be1f-a82b5834f728"
 					(reference "#PWR012")
@@
 		)
 		(instances
-			(project "mls12"
+			(project "mls25"
 				(path "/53bda2f8-fdf0-44f4-aced-3b46017d299c/9f8390ae-91ea-4278-be1f-a82b5834f728"
 					(reference "FB5")
@@
 		)
 		(instances
-			(project "mls12"
+			(project "mls25"
 				(path "/53bda2f8-fdf0-44f4-aced-3b46017d299c/9f8390ae-91ea-4278-be1f-a82b5834f728"
 					(reference "FB6")
@@
 		)
 		(instances
-			(project "mls12"
+			(project "mls25"
 				(path "/53bda2f8-fdf0-44f4-aced-3b46017d299c/9f8390ae-91ea-4278-be1f-a82b5834f728"
 					(reference "FB4")
@@
 		)
 		(instances
-			(project "mls12"
+			(project "mls25"
 				(path "/53bda2f8-fdf0-44f4-aced-3b46017d299c/9f8390ae-91ea-4278-be1f-a82b5834f728"
 					(reference "C6")
@@
 		)
 		(instances
-			(project "mls12"
+			(project "mls25"
 				(path "/53bda2f8-fdf0-44f4-aced-3b46017d299c/9f8390ae-91ea-4278-be1f-a82b5834f728"
 					(reference "TP5")
@@
 		)
 		(instances
-			(project "mls12"
+			(project "mls25"
 				(path "/53bda2f8-fdf0-44f4-aced-3b46017d299c/9f8390ae-91ea-4278-be1f-a82b5834f728"
 					(reference "C4")
@@
 	)
 	(symbol
-		(lib_id "mls12:Ag5724-LPB")
+		(lib_id "mls25:Ag5724-LPB")
 		(at 166.37 102.87 0)
 		(unit 1)
@@
 			)
 		)
-		(property "Footprint" "mls12:Ag5724-LPB"
+		(property "Footprint" "mls25:Ag5724-LPB"
 			(at 166.37 102.87 0)
 			(effects
@@
 			)
 		)
-		(property "Footprint" "mls12:DPC817S-C-TR"
+		(property "Footprint" "mls25:DPC817S-C-TR"
 			(at 161.29 72.39 0)
 			(effects
@@
 		)
 		(instances
-			(project "mls12"
+			(project "mls25"
 				(path "/53bda2f8-fdf0-44f4-aced-3b46017d299c/9f8390ae-91ea-4278-be1f-a82b5834f728"
 					(reference "FB1")
@@
 		)
 		(instances
-			(project "mls12"
+			(project "mls25"
 				(path "/53bda2f8-fdf0-44f4-aced-3b46017d299c/9f8390ae-91ea-4278-be1f-a82b5834f728"
 					(reference "#PWR010")
@@
 		)
 		(instances
-			(project "mls12"
+			(project "mls25"
 				(path "/53bda2f8-fdf0-44f4-aced-3b46017d299c/9f8390ae-91ea-4278-be1f-a82b5834f728"
 					(reference "#PWR084")
@@
 		)
 		(instances
-			(project "mls12"
+			(project "mls25"
 				(path "/53bda2f8-fdf0-44f4-aced-3b46017d299c/9f8390ae-91ea-4278-be1f-a82b5834f728"
 					(reference "#PWR08")
@@
 		)
 		(instances
-			(project "mls12"
+			(project "mls25"
 				(path "/53bda2f8-fdf0-44f4-aced-3b46017d299c/9f8390ae-91ea-4278-be1f-a82b5834f728"
 					(reference "C5")
@@
 		)
 		(instances
-			(project "mls12"
+			(project "mls25"
 				(path "/53bda2f8-fdf0-44f4-aced-3b46017d299c/9f8390ae-91ea-4278-be1f-a82b5834f728"
 					(reference "#PWR078")
@@
 		)
 		(instances
-			(project "mls12"
+			(project "mls25"
 				(path "/53bda2f8-fdf0-44f4-aced-3b46017d299c/9f8390ae-91ea-4278-be1f-a82b5834f728"
 					(reference "TP33")
@@
 		)
 		(instances
-			(project "mls12"
+			(project "mls25"
 				(path "/53bda2f8-fdf0-44f4-aced-3b46017d299c/9f8390ae-91ea-4278-be1f-a82b5834f728"
 					(reference "#PWR011")
@@
 		)
 		(instances
-			(project "mls12"
+			(project "mls25"
 				(path "/53bda2f8-fdf0-44f4-aced-3b46017d299c/9f8390ae-91ea-4278-be1f-a82b5834f728"
 					(reference "FB2")
@@
 		)
 		(instances
-			(project "mls12"
+			(project "mls25"
 				(path "/53bda2f8-fdf0-44f4-aced-3b46017d299c/9f8390ae-91ea-4278-be1f-a82b5834f728"
 					(reference "TP6")
@@
 		)
 		(instances
-			(project "mls12"
+			(project "mls25"
 				(path "/53bda2f8-fdf0-44f4-aced-3b46017d299c/9f8390ae-91ea-4278-be1f-a82b5834f728"
 					(reference "C7")
@@
 		)
 		(instances
-			(project "mls12"
+			(project "mls25"
 				(path "/53bda2f8-fdf0-44f4-aced-3b46017d299c/9f8390ae-91ea-4278-be1f-a82b5834f728"
 					(reference "C10")
@@
 	)
 	(symbol
-		(lib_id "mls12:LMB110S-TP")
+		(lib_id "mls25:LMB110S-TP")
 		(at 68.58 109.22 0)
 		(unit 1)
@@
 			)
 		)
-		(property "Footprint" "mls12:LMB110S-TP"
+		(property "Footprint" "mls25:LMB110S-TP"
 			(at 72.39 106.045 0)
 			(effects
@@
 		)
 		(instances
-			(project "mls12"
+			(project "mls25"
 				(path "/53bda2f8-fdf0-44f4-aced-3b46017d299c/9f8390ae-91ea-4278-be1f-a82b5834f728"
 					(reference "D4")
@@
 		)
 		(instances
-			(project "mls12"
+			(project "mls25"
 				(path "/53bda2f8-fdf0-44f4-aced-3b46017d299c/9f8390ae-91ea-4278-be1f-a82b5834f728"
 					(reference "#PWR076")
@@
 		)
 		(instances
-			(project "mls12"
+			(project "mls25"
 				(path "/53bda2f8-fdf0-44f4-aced-3b46017d299c/9f8390ae-91ea-4278-be1f-a82b5834f728"
 					(reference "#PWR07")
@@
 		)
 		(instances
-			(project "mls12"
+			(project "mls25"
 				(path "/53bda2f8-fdf0-44f4-aced-3b46017d299c/9f8390ae-91ea-4278-be1f-a82b5834f728"
 					(reference "TP4")
@@
 		)
 		(instances
-			(project "mls12"
+			(project "mls25"
 				(path "/53bda2f8-fdf0-44f4-aced-3b46017d299c/9f8390ae-91ea-4278-be1f-a82b5834f728"
 					(reference "C8")
@@
 		)
 		(instances
-			(project "mls12"
+			(project "mls25"
 				(path "/53bda2f8-fdf0-44f4-aced-3b46017d299c/9f8390ae-91ea-4278-be1f-a82b5834f728"
 					(reference "FB3")

Commit message: Exclude test pads from BOM
Parts:
- TP1, TP33, TP4, TP5, TP6, TP7, TP8: now left out of the parts list
Changed lines of the file:
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@@
 		(unit 1)
 		(exclude_from_sim no)
-		(in_bom yes)
+		(in_bom no)
 		(on_board yes)
 		(dnp no)
@@
 		(unit 1)
 		(exclude_from_sim no)
-		(in_bom yes)
+		(in_bom no)
 		(on_board yes)
 		(dnp no)
@@
 		(unit 1)
 		(exclude_from_sim no)
-		(in_bom yes)
+		(in_bom no)
 		(on_board yes)
 		(dnp no)
@@
 		(unit 1)
 		(exclude_from_sim no)
-		(in_bom yes)
+		(in_bom no)
 		(on_board yes)
 		(dnp no)
@@
 		(unit 1)
 		(exclude_from_sim no)
-		(in_bom yes)
+		(in_bom no)
 		(on_board yes)
 		(dnp no)
@@
 		(unit 1)
 		(exclude_from_sim no)
-		(in_bom yes)
+		(in_bom no)
 		(on_board yes)
 		(dnp no)
@@
 		(unit 1)
 		(exclude_from_sim no)
-		(in_bom yes)
+		(in_bom no)
 		(on_board yes)
 		(dnp no)
