File: pcb/mls25_led_output.kicad_sch (KiCad schematic)
At the start: 21 parts, among them J4 JST B3B-ZR, J5 DC barrel plug, Q1 DMG3406L, Q2 DMG3406L

Commit message: Rename `mls12` to `mls25`
Module output was changed from 12W to 25W during the course of development.
Update filenames to reflect that.
Parts:
- F1: footprint mls12:SMD1812B050TF_30 -> mls25:SMD1812B050TF_30
- J5: footprint mls12:DC_Barrel_Plug_2.1x5.5mm -> mls25:DC_Barrel_Plug_2.1x5.5mm
Changed lines of the file:
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@@
 		)
 		(instances
-			(project "mls12"
+			(project "mls25"
 				(path "/53bda2f8-fdf0-44f4-aced-3b46017d299c/643c732c-b7d6-4ad7-813b-2f70dd62e640"
 					(reference "R40")
@@
 		)
 		(instances
-			(project "mls12"
+			(project "mls25"
 				(path "/53bda2f8-fdf0-44f4-aced-3b46017d299c/643c732c-b7d6-4ad7-813b-2f70dd62e640"
 					(reference "TP26")
@@
 		)
 		(instances
-			(project "mls12"
+			(project "mls25"
 				(path "/53bda2f8-fdf0-44f4-aced-3b46017d299c/643c732c-b7d6-4ad7-813b-2f70dd62e640"
 					(reference "R41")
@@
 			)
 		)
-		(property "Footprint" "mls12:SMD1812B050TF_30"
+		(property "Footprint" "mls25:SMD1812B050TF_30"
 			(at 86.36 46.99 0)
 			(effects
@@
 		)
 		(instances
-			(project "mls12"
+			(project "mls25"
 				(path "/53bda2f8-fdf0-44f4-aced-3b46017d299c/643c732c-b7d6-4ad7-813b-2f70dd62e640"
 					(reference "D8")
@@
 		)
 		(instances
-			(project "mls12"
+			(project "mls25"
 				(path "/53bda2f8-fdf0-44f4-aced-3b46017d299c/643c732c-b7d6-4ad7-813b-2f70dd62e640"
 					(reference "TP25")
@@
 		)
 		(instances
-			(project "mls12"
+			(project "mls25"
 				(path "/53bda2f8-fdf0-44f4-aced-3b46017d299c/643c732c-b7d6-4ad7-813b-2f70dd62e640"
 					(reference "#PWR059")
@@
 		)
 		(instances
-			(project "mls12"
+			(project "mls25"
 				(path "/53bda2f8-fdf0-44f4-aced-3b46017d299c/643c732c-b7d6-4ad7-813b-2f70dd62e640"
 					(reference "J4")
@@
 		)
 		(instances
-			(project "mls12"
+			(project "mls25"
 				(path "/53bda2f8-fdf0-44f4-aced-3b46017d299c/643c732c-b7d6-4ad7-813b-2f70dd62e640"
 					(reference "#PWR060")
@@
 		)
 		(instances
-			(project "mls12"
+			(project "mls25"
 				(path "/53bda2f8-fdf0-44f4-aced-3b46017d299c/643c732c-b7d6-4ad7-813b-2f70dd62e640"
 					(reference "#PWR062")
@@
 		)
 		(instances
-			(project "mls12"
+			(project "mls25"
 				(path "/53bda2f8-fdf0-44f4-aced-3b46017d299c/643c732c-b7d6-4ad7-813b-2f70dd62e640"
 					(reference "#PWR080")
@@
 		)
 		(instances
-			(project "mls12"
+			(project "mls25"
 				(path "/53bda2f8-fdf0-44f4-aced-3b46017d299c/643c732c-b7d6-4ad7-813b-2f70dd62e640"
 					(reference "R38")
@@
 		)
 		(instances
-			(project "mls12"
+			(project "mls25"
 				(path "/53bda2f8-fdf0-44f4-aced-3b46017d299c/643c732c-b7d6-4ad7-813b-2f70dd62e640"
 					(reference "#PWR061")
@@
 		)
 		(instances
-			(project "mls12"
+			(project "mls25"
 				(path "/53bda2f8-fdf0-44f4-aced-3b46017d299c/643c732c-b7d6-4ad7-813b-2f70dd62e640"
 					(reference "#PWR063")
@@
 		)
 		(instances
-			(project "mls12"
+			(project "mls25"
 				(path "/53bda2f8-fdf0-44f4-aced-3b46017d299c/643c732c-b7d6-4ad7-813b-2f70dd62e640"
 					(reference "#PWR057")
@@
 		)
 		(instances
-			(project "mls12"
+			(project "mls25"
 				(path "/53bda2f8-fdf0-44f4-aced-3b46017d299c/643c732c-b7d6-4ad7-813b-2f70dd62e640"
 					(reference "#PWR056")
@@
 		)
 		(instances
-			(project "mls12"
+			(project "mls25"
 				(path "/53bda2f8-fdf0-44f4-aced-3b46017d299c/643c732c-b7d6-4ad7-813b-2f70dd62e640"
 					(reference "C39")
@@
 		)
 		(instances
-			(project "mls12"
+			(project "mls25"
 				(path "/53bda2f8-fdf0-44f4-aced-3b46017d299c/643c732c-b7d6-4ad7-813b-2f70dd62e640"
 					(reference "#PWR058")
@@
 		)
 		(instances
-			(project "mls12"
+			(project "mls25"
 				(path "/53bda2f8-fdf0-44f4-aced-3b46017d299c/643c732c-b7d6-4ad7-813b-2f70dd62e640"
 					(reference "#PWR065")
@@
 			)
 		)
-		(property "Footprint" "mls12:DC_Barrel_Plug_2.1x5.5mm"
+		(property "Footprint" "mls25:DC_Barrel_Plug_2.1x5.5mm"
 			(at 232.41 96.52 0)
 			(effects
@@
 		)
 		(instances
-			(project "mls12"
+			(project "mls25"
 				(path "/53bda2f8-fdf0-44f4-aced-3b46017d299c/643c732c-b7d6-4ad7-813b-2f70dd62e640"
 					(reference "R39")
@@
 		)
 		(instances
-			(project "mls12"
+			(project "mls25"
 				(path "/53bda2f8-fdf0-44f4-aced-3b46017d299c/643c732c-b7d6-4ad7-813b-2f70dd62e640"
 					(reference "#PWR064")
@@
 		)
 		(instances
-			(project "mls12"
+			(project "mls25"
 				(path "/53bda2f8-fdf0-44f4-aced-3b46017d299c/643c732c-b7d6-4ad7-813b-2f70dd62e640"
 					(reference "TP29")
@@
 		)
 		(instances
-			(project "mls12"
+			(project "mls25"
 				(path "/53bda2f8-fdf0-44f4-aced-3b46017d299c/643c732c-b7d6-4ad7-813b-2f70dd62e640"
 					(reference "R45")
@@
 		)
 		(instances
-			(project "mls12"
+			(project "mls25"
 				(path "/53bda2f8-fdf0-44f4-aced-3b46017d299c/643c732c-b7d6-4ad7-813b-2f70dd62e640"
 					(reference "Q2")
@@
 		)
 		(instances
-			(project "mls12"
+			(project "mls25"
 				(path "/53bda2f8-fdf0-44f4-aced-3b46017d299c/643c732c-b7d6-4ad7-813b-2f70dd62e640"
 					(reference "R37")
@@
 		)
 		(instances
-			(project "mls12"
+			(project "mls25"
 				(path "/53bda2f8-fdf0-44f4-aced-3b46017d299c/643c732c-b7d6-4ad7-813b-2f70dd62e640"
 					(reference "R46")
@@
 		)
 		(instances
-			(project "mls12"
+			(project "mls25"
 				(path "/53bda2f8-fdf0-44f4-aced-3b46017d299c/643c732c-b7d6-4ad7-813b-2f70dd62e640"
 					(reference "R44")
@@
 		)
 		(instances
-			(project "mls12"
+			(project "mls25"
 				(path "/53bda2f8-fdf0-44f4-aced-3b46017d299c/643c732c-b7d6-4ad7-813b-2f70dd62e640"
 					(reference "R42")

Commit message: Change output polyfuse from 500mA to 750mA
Parts:
- F1: value 500mA/30V -> 750mA/24V; MPN SMD1812B050TF/30 -> SMD1812B075TF/24
Changed lines of the file:
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@@
 			)
 		)
-		(property "Value" "500mA/30V"
+		(property "Value" "750mA/24V"
 			(at 91.44 41.91 90)
 			(effects
@@
 			)
 		)
-		(property "MPN" "SMD1812B050TF/30"
+		(property "MPN" "SMD1812B075TF/24"
 			(at 91.44 45.72 0)
 			(effects

Commit message: Exclude test pads from BOM
Parts:
- J5, TP25, TP26, TP29: now left out of the parts list
Changed lines of the file:
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@@
 		(unit 1)
 		(exclude_from_sim no)
-		(in_bom yes)
+		(in_bom no)
 		(on_board yes)
 		(dnp no)
@@
 		(unit 1)
 		(exclude_from_sim no)
-		(in_bom yes)
+		(in_bom no)
 		(on_board yes)
 		(dnp no)
@@
 		(unit 1)
 		(exclude_from_sim no)
-		(in_bom yes)
+		(in_bom no)
 		(on_board yes)
 		(dnp no)
@@
 		(unit 1)
 		(exclude_from_sim no)
-		(in_bom yes)
-		(on_board yes)
-		(dnp no)
+		(in_bom no)
+		(on_board yes)
+		(dnp no)
