File: pcb/mls25_mcu.kicad_sch (KiCad schematic)
At the start: 48 parts, among them J2 TC2070-FP, J3 SM04B-SRSS-TB, U4 STM32H563RIT6, Y2 25MHz

Commit message: Rename `mls12` to `mls25`
Module output was changed from 12W to 25W during the course of development.
Update filenames to reflect that.
Parts:
- J2: symbol mls12:TC2070-Contecto -> mls25:TC2070-Contecto
- U4: symbol mls12:STM32H563RIT6 -> mls25:STM32H563RIT6

Commit message: Fix ERC warnings/errors
*  Add NC-flags to microcontroller pins.
*  Fix STM32 VCAP, ~RESET pin type.
*  Add PWR_FLAG symbols.
Parts:
- J2: MF (none) -> TagConnect; MPN (none) -> TC2070-IDC-FP
Connections:
- no-connect marks 0 -> 17
Changed lines of the file:
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@@
 	(title_block
 		(title "Microcontroller")
-		(date "2025-07-26")
+		(date "2025-09-27")
 		(rev "A")
 		(company "Quomodo BV")
@@
 		(color 0 0 0 0)
 	)
+	(no_connect
+		(at 237.49 191.77)
+	)
+	(no_connect
+		(at 351.79 66.04)
+	)
+	(no_connect
+		(at 86.36 185.42)
+	)
+	(no_connect
+		(at 163.83 218.44)
+	)
+	(no_connect
+		(at 86.36 210.82)
+	)
+	(no_connect
+		(at 237.49 201.93)
+	)
+	(no_connect
+		(at 163.83 220.98)
+	)
+	(no_connect
+		(at 237.49 184.15)
+	)
+	(no_connect
+		(at 237.49 252.73)
+	)
+	(no_connect
+		(at 163.83 185.42)
+	)
+	(no_connect
+		(at 86.36 223.52)
+	)
+	(no_connect
+		(at 237.49 204.47)
+	)
+	(no_connect
+		(at 86.36 208.28)
+	)
+	(no_connect
+		(at 163.83 187.96)
+	)
+	(no_connect
+		(at 86.36 195.58)
+	)
+	(no_connect
+		(at 237.49 219.71)
+	)
+	(no_connect
+		(at 237.49 212.09)
+	)
 	(bus_entry
 		(at 186.69 187.96)
@@
 	)
 	(symbol
+		(lib_id "power:PWR_FLAG")
+		(at 27.94 40.64 90)
+		(unit 1)
+		(exclude_from_sim no)
+		(in_bom yes)
+		(on_board yes)
+		(dnp no)
+		(fields_autoplaced yes)
+		(property "Reference" "#FLG02"
+			(at 26.035 40.64 0)
+			(effects
+				(font
+					(size 1.27 1.27)
+				)
+				(hide yes)
+			)
+		)
+		(property "Value" "PWR_FLAG"
+			(at 24.13 40.6399 90)
+			(effects
+				(font
+					(size 1.27 1.27)
+				)
+				(justify left)
+				(hide yes)
+			)
+		)
+		(property "Footprint" ""
+			(at 27.94 40.64 0)
+			(effects
+				(font
+					(size 1.27 1.27)
+				)
+				(hide yes)
+			)
+		)
+		(property "Datasheet" "~"
+			(at 27.94 40.64 0)
+			(effects
+				(font
+					(size 1.27 1.27)
+				)
+				(hide yes)
+			)
+		)
+		(property "Description" "Special symbol for telling ERC where power comes from"
+			(at 27.94 40.64 0)
+			(effects
+				(font
+					(size 1.27 1.27)
+				)
+				(hide yes)
+			)
+		)
+		(property "MF" ""
+			(at 27.94 40.64 0)
+			(effects
+				(font
+					(size 1.27 1.27)
+				)
+				(hide yes)
+			)
+		)
+		(property "MPN" ""
+			(at 27.94 40.64 0)
+			(effects
+				(font
+					(size 1.27 1.27)
+				)
+				(hide yes)
+			)
+		)
+		(pin "1"
+		)
+		(instances
+			(project ""
+				(path "/53bda2f8-fdf0-44f4-aced-3b46017d299c/302b6a68-f945-4d74-bd08-29eb164cd442"
+					(reference "#FLG02")
+					(unit 1)
+				)
+			)
+		)
+	)
+	(symbol
 		(lib_id "Connector:TestPoint")
 		(at 367.03 135.89 0)
@@
 			)
 		)
+		(property "MF" "TagConnect"
+			(at 364.49 62.23 0)
+			(effects
+				(font
+					(size 1.27 1.27)
+				)
+				(hide yes)
+			)
+		)
+		(property "MPN" "TC2070-IDC-FP"
+			(at 364.49 62.23 0)
+			(effects
+				(font
+					(size 1.27 1.27)
+				)
+				(hide yes)
+			)
+		)
 		(pin "9"
 		)
@@
 	)
 	(symbol
+		(lib_name "STM32H563RIT6_1")
 		(lib_id "mls25:STM32H563RIT6")
 		(at 140.97 62.23 0)
@@
 		)
 		(pin "17"
-			(alternate "PA3_ADC1_INP15")
 		)
 		(instances
@@
 	)
 	(symbol
+		(lib_name "STM32H563RIT6_3")
 		(lib_id "mls25:STM32H563RIT6")
 		(at 149.86 204.47 0)
@@
 		)
 		(pin "17"
-			(alternate "PA3_ADC1_INP15")
 		)
 		(instances
@@
 		)
 		(pin "17"
-			(alternate "PA3_ADC1_INP15")
 		)
 		(instances
@@
 	)
 	(symbol
+		(lib_name "STM32H563RIT6_2")
 		(lib_id "mls25:STM32H563RIT6")
 		(at 72.39 204.47 0)
@@
 	)
 	(symbol
+		(lib_name "STM32H563RIT6_4")
 		(lib_id "mls25:STM32H563RIT6")
 		(at 223.52 203.2 0)
@@
 		)
 		(pin "17"
-			(alternate "PA3_ADC1_INP15")
 		)
 		(instances
@@
 	)
 	(symbol
+		(lib_name "STM32H563RIT6_5")
 		(lib_id "mls25:STM32H563RIT6")
 		(at 223.52 252.73 0)
@@
 		)
 		(pin "17"
-			(alternate "PA3_ADC1_INP15")
 		)
 		(instances

Commit message: Tweaks/fixes after design review
*  Fix RJ45 refdes on silkscreen.
*  Change PHY IRQ pullup from 1K to 4K7 per datasheet recommendations.
*  Add skew correction on MDI TX differential pair.
*  Remove copper under magnetics.
*  Add annotation that TYP2_DET signal requires MCU internal pullup.
Other:
- note added: "DET: active-low, internal pull-up"
Changed lines of the file:
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@@
+		)
+	)
+	(text "DET: active-low,\ninternal pull-up"
+		(exclude_from_sim no)
+		(at 275.59 217.17 0)
+		(effects
+			(font
+				(size 1.27 1.27)
+			)
+			(justify left)
 		)
 	)

Commit message: Exclude test pads from BOM
Parts:
- TP14, TP15, TP16, TP17, TP18, TP19, TP20, TP21, TP22, TP23, TP24: now left out of the parts list
Changed lines of the file:
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@@
 		(unit 1)
 		(exclude_from_sim no)
-		(in_bom yes)
+		(in_bom no)
 		(on_board yes)
 		(dnp no)
@@
 		(unit 1)
 		(exclude_from_sim no)
-		(in_bom yes)
+		(in_bom no)
 		(on_board yes)
 		(dnp no)
@@
 		(unit 1)
 		(exclude_from_sim no)
-		(in_bom yes)
+		(in_bom no)
 		(on_board yes)
 		(dnp no)
@@
 		(unit 1)
 		(exclude_from_sim no)
-		(in_bom yes)
+		(in_bom no)
 		(on_board yes)
 		(dnp no)
@@
 		(unit 1)
 		(exclude_from_sim no)
-		(in_bom yes)
+		(in_bom no)
 		(on_board yes)
 		(dnp no)
@@
 		(unit 1)
 		(exclude_from_sim no)
-		(in_bom yes)
+		(in_bom no)
 		(on_board yes)
 		(dnp no)
@@
 		(unit 1)
 		(exclude_from_sim no)
-		(in_bom yes)
+		(in_bom no)
 		(on_board yes)
 		(dnp no)
@@
 		(unit 1)
 		(exclude_from_sim no)
-		(in_bom yes)
+		(in_bom no)
 		(on_board yes)
 		(dnp no)
@@
 		(unit 1)
 		(exclude_from_sim no)
-		(in_bom yes)
+		(in_bom no)
 		(on_board yes)
 		(dnp no)
@@
 		(unit 1)
 		(exclude_from_sim no)
-		(in_bom yes)
+		(in_bom no)
 		(on_board yes)
 		(dnp no)
@@
 		(unit 1)
 		(exclude_from_sim no)
-		(in_bom yes)
+		(in_bom no)
 		(on_board yes)
 		(dnp no)
