File: pcb/mls25_nor_flash.kicad_sch (KiCad schematic)
At the start: 4 parts, among them U5 W25Q16JVSS

Commit message: Exclude test pads from BOM
Parts:
- TP32: now left out of the parts list
Changed lines of the file:
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@@
 		(unit 1)
 		(exclude_from_sim no)
-		(in_bom yes)
+		(in_bom no)
 		(on_board yes)
 		(dnp no)
